File: kicad/pb3-replacement.kicad_sch (KiCad schematic)
At the start: 0 parts

Commit message: test
Parts:
- added BT1: LiFePO4_1500mAh, symbol Device:Battery_Cell
- added C4, C5: 22uF, Capacitor_SMD:C_1206_3216Metric, symbol Device:C
- added D1: CHRG, LED_SMD:LED_0603_1608Metric, symbol Device:LED
- added D2: FULL, LED_SMD:LED_0603_1608Metric, symbol Device:LED
- added D3: SS34, Diode_SMD:D_SMA, symbol Device:D_Schottky
- added J1: USB_C, Connector_USB:USB_C_Receptacle_GCT_USB4105-xx-A, symbol Connector:USB_C_Receptacle_USB2.0
- added J2: DECK_5V, Connector_PinHeader_2.54mm:PinHeader_1x02_P2.54mm_Vertical, symbol Connector:Conn_01x02_Pin
- added L1: 22uH, Inductor_SMD:L_7.3x7.3_H3.5, symbol Device:L
- added Q1: FS8205A, Package_TO_SOT_SMD:SOT-23-6, symbol Transistor_FET:FS8205A
- added R5: 10k, Resistor_SMD:R_0603_1608Metric, symbol Device:R
- added R6: 15k, Resistor_SMD:R_0603_1608Metric, symbol Device:R
- added U1: CN3058E, Package_SO:SOP-8_3.9x4.9mm_P1.27mm_EP, symbol Regulator_Switching:CN3058E
- added U2: HY2112, Package_TO_SOT_SMD:SOT-23-6, symbol Power_Protection:HY2112
- added U3: MT3608, Package_TO_SOT_SMD:SOT-23-6, symbol Regulator_Switching:MT3608
Other:
- note added: "CN3058E LiFePO4 Charger"
- note added: "HY2112 + FS8205 1S BMS"
- note added: "LiFePO4 1500mAh 3.2V nom"
- note added: "MT3608 Boost 5V"
- note added: "TO DECK"
- note added: "USB-C 5V IN"
- note removed: "Host deck: HS-PC202MII. Wall wart + OEM pack missing. Dimensions from measurement photos + Stereo2Go thread."
- title: PB-3 Replacement -> PB-3 LiFePO4 Replacement

Commit message: pre cleanup
Parts:
- removed C4, C5: 22uF, Capacitor_SMD:C_1206_3216Metric, symbol Device:C
- removed D2: FULL, LED_SMD:LED_0603_1608Metric, symbol Device:LED
- removed D3: SS34, Diode_SMD:D_SMA, symbol Device:D_Schottky
- BT1: value LiFePO4_1500mAh -> LiPo_3.7V
- D1: renamed from L1; value 22uH -> 2.7V_Zener; footprint Inductor_SMD:L_7.3x7.3_H3.5 -> Diode_SMD:D_SOD-123; symbol Device:L -> Device:D_Zener; LCSC C334097 -> (none)
- D2: renamed from R6; value 15k -> CHRG; footprint Resistor_SMD:R_0603_1608Metric -> LED_SMD:LED_0603_1608Metric; symbol Device:R -> Device:LED
- D3: renamed from J2; value DECK_5V -> FULL; footprint Connector_PinHeader_2.54mm:PinHeader_1x02_P2.54mm_Vertical -> LED_SMD:LED_0603_1608Metric; symbol Connector:Conn_01x02_Pin -> Device:LED
- J2: renamed from R5; value 10k -> DECK_2.4V; footprint Resistor_SMD:R_0603_1608Metric -> Connector_PinHeader_2.54mm:PinHeader_1x02_P2.54mm_Vertical; symbol Device:R -> Connector:Conn_01x02_Pin
- Q1: LCSC C32254 -> C16052
- R1: renamed from D1; value CHRG -> 100k; footprint LED_SMD:LED_0603_1608Metric -> Resistor_SMD:R_0603_1608Metric; symbol Device:LED -> Device:R
- U1: value CN3058E -> TP4056; footprint Package_SO:SOP-8_3.9x4.9mm_P1.27mm_EP -> Package_SO:SOP-8_3.9x4.9mm_P1.27mm; symbol Regulator_Switching:CN3058E -> Battery_Management:TP4056; LCSC C112011 -> C16581
- U2: value HY2112 -> DW01A; symbol Power_Protection:HY2112 -> Battery_Management:DW01A; LCSC C161942 -> C351410
- U3: value MT3608 -> Buck_2.4V; footprint Package_TO_SOT_SMD:SOT-23-6 -> Package_TO_SOT_SMD:SOT-23-5; symbol Regulator_Switching:MT3608 -> Regulator_Switching:TPS62200; LCSC C84817 -> (none)
Other:
- note added: "Buck 3.7V->2.4V"
- note added: "DECK 2.4V"
- note added: "DW01A + FS8205 1S BMS OV/UV/OC"
- note added: "LiPo 500-1500mAh 3.7V nom"
- note added: "OVP Zener/TVS <3V clamp"
- note added: "OVP: Clamps output if buck MOSFET shorts Protects deck from 3.7V"
- note added: "Rfb: 100k=2.4V 120k=2.1V"
- note added: "TP4056 LiPo Charger 4.2V CC/CV"
- note removed: "CN3058E LiFePO4 Charger"
- note removed: "HY2112 + FS8205 1S BMS"
- note removed: "LiFePO4 1500mAh 3.2V nom"
- note removed: "MT3608 Boost 5V"
- note removed: "TO DECK"
- title: PB-3 LiFePO4 Replacement -> PB-3 LiPo Replacement

Commit message: cleanup
Other:
- note added: "Buck 3.7V->2.0V"
- note added: "DECK 2.0V"
- note removed: "Buck 3.7V->2.4V"
- note removed: "DECK 2.4V"
Changed lines of the file:
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@@
     (rev "0.4")
     (company "AIWA HS-PC202MII")
-    (comment 1 "LiPo 3.7V + Buck 2.4V + OVP")
+    (comment 1 "LiPo 3.7V + Buck 2.0V + OVP")
     (comment 2 "Open source - CC BY-SA 4.0")
   )
@@
     (effects (font (size 2.54 2.54)) (justify left))
   )
-  (text "Buck\n3.7V->2.4V" (at 157.48 50.8 0)
+  (text "Buck\n3.7V->2.0V" (at 157.48 50.8 0)
     (effects (font (size 2.54 2.54)) (justify left))
   )
@@
     (effects (font (size 2.54 2.54)) (justify left))
   )
-  (text "DECK\n2.4V" (at 233.68 50.8 0)
+  (text "DECK\n2.0V" (at 233.68 50.8 0)
     (effects (font (size 2.54 2.54)) (justify left))
   )
