File: kicad/pb3-replacement.kicad_sch (KiCad schematic)
At the start: 11 parts, among them J1 USB_C, J2 DECK_2.4V, Q1 FS8205A, U1 TP4056, U2 DW01A, U3 Buck_2.4V

Commit message: Wire pb3-replacement schematic with real symbols, unblock Stage 2 netlist export
Co-authored-by: donnels <14863623+donnels@users.noreply.github.com>
Parts:
- removed J1: USB_C, Connector_USB:USB_C_Receptacle_GCT_USB4105-xx-A, symbol Connector:USB_C_Receptacle_USB2.0
- removed Q1: FS8205A, Package_TO_SOT_SMD:SOT-23-6, symbol Transistor_FET:FS8205A
- removed U1: TP4056, Package_SO:SOP-8_3.9x4.9mm_P1.27mm, symbol Battery_Management:TP4056
- removed U3: Buck_2.4V, Package_TO_SOT_SMD:SOT-23-5, symbol Regulator_Switching:TPS62200
- added C1: 10uF, Capacitor_SMD:C_0603_1608Metric, symbol Device:C
- added J1: USB_C, Connector_USB:USB_C_Receptacle_GCT_USB4105-xx-A, symbol Connector:USB_C_Receptacle_PowerOnly_6P
- added L1: 2.2uH, Inductor_SMD:L_0805_2012Metric, symbol Device:L
- added Q1: FS8205A, Package_TO_SOT_SMD:SOT-23-6, symbol Transistor_FET:DMG9926UDM
- added R2: 2.4k, Resistor_SMD:R_0603_1608Metric, symbol Device:R
- added R3, R4: 1k, Resistor_SMD:R_0603_1608Metric, symbol Device:R
- added R5: TBD, Resistor_SMD:R_0603_1608Metric, symbol Device:R
- added U1: TP4056, Package_SO:SOP-8_3.9x4.9mm_P1.27mm, symbol Battery_Management:TP4056-42-ESOP8
- added U3: Buck_2.0V, Package_TO_SOT_SMD:SOT-23-5, symbol Regulator_Switching:TPS62200DBV
- J2: value DECK_2.4V -> DECK_2.0V
Connections:
- net GND: now also D1.2 (A), J2.2 (Pin_2), U2.2 (CS), U2.6 (GND), C1.2, J1.A12 (GND), J1.B12 (GND), J1.S1 (SHIELD), Q1.2 (S1/D2), Q1.3 (S2), Q1.5 (S1/D2), R2.2, R5.2, U1.1 (TEMP), U1.3 (GND), U1.8 (CE), U1.9 (EPAD), U3.2 (GND)
- net VBAT: now also BT1.1 (+), U2.5 (VCC), U1.5 (BAT), U3.1 (VI), U3.3 (EN)
- net VBUS: now also J1.A9 (VBUS), J1.B9 (VBUS), R3.1, R4.1, U1.4 (V_{CC})
- net VOUT: now also D1.1 (K), J2.1 (Pin_1), R1.1, C1.1, L1.2
- new net CHRG: D2.1 (K), U1.7 (~{CHRG})
- new net CHRG_A: D2.2 (A), R3.2
- new net FB: R1.2, R5.1, U3.4 (FB)
- new net NC_CC1: J1.A5 (CC1)
- new net NC_CC2: J1.B5 (CC2)
- new net NC_TD: U2.4 (TD)
- new net OC: Q1.4 (G2), U2.3 (OC)
- new net OD: Q1.6 (G1), U2.1 (OD)
- new net PROG: R2.1, U1.2 (PROG)
- new net STDBY: D3.1 (K), U1.6 (~{STDBY})
- new net STDBY_A: D3.2 (A), R4.2
- new net SW: L1.1, U3.5 (SW)
- new net VBAT_RAW_NEG: BT1.2 (-), Q1.1 (D1)
Other:
- note removed: "Buck 3.7V->2.0V"
- note removed: "DECK 2.0V"
- note removed: "DW01A + FS8205 1S BMS OV/UV/OC"
- note removed: "LiPo 500-1500mAh 3.7V nom"
- note removed: "OVP Zener/TVS <3V clamp"
- note removed: "OVP: Clamps output if buck MOSFET shorts Protects deck from 3.7V"
- note removed: "Rfb: 100k=2.4V 120k=2.1V"
- note removed: "TP4056 LiPo Charger 4.2V CC/CV"
- note removed: "USB-C 5V IN"
